File: kicad/solderbit-gamepad.kicad_pcb (KiCad board)
At the start: 2 copper layers, 114.5 x 45 mm, 47 parts, among them SW1 DPDT, U1 Shift_Register_74HC165D

Commit message: KiCad font fixes and 3D renders
Parts:
- removed ?: , clipboard:2530302b-2469-4c92-a02c-03a2972aa858
- removed ?: , clipboard:7ef0c00c-865a-4d4a-b67e-d24925b7692a
- removed ?: , clipboard:eb6b9f81-2bd5-4935-ac84-cf1cb09f0a3b
- removed ?: , clipboard:f35a52af-685d-4dbc-bad2-5c89170f1274
- removed ?: , clipboard:d516af6b-2eaf-415c-a72b-82543e7ff2ee
- removed ?: , clipboard:447a6eb8-5143-46bc-a893-9c0e9147b170
- removed ?: , clipboard:4f59e82c-baf0-4beb-a700-d93e24cfaf47
- removed ?: , clipboard:3a223a59-e2f8-418b-9e6a-e43a3431079a
- removed C2, C3, C4, C5, C6: 1uF, Solderbit_Gamepad:1206_Capacitor
- removed D1, D2, D3, D4, D5: NeoPixel_WS2812B, Solderbit_Gamepad:NeoPixel_WS2812B
- removed R9: 300Ω, Solderbit_Gamepad:1206_Resistor
- BT1: value Battery -> BH-AAA-B5AA001
- D6: value D_Schottky -> BAT60B
- J1: value ~ -> Microbit
- S1, S2, S3, S4, S5, S6: value ~ -> TS-1002S-AR06026
- S7, S8: value SW_Push -> TS-1037-A4B3-D2
- SW1: value DPDT -> MST22D18G2 125
- U1: value Shift_Register_74HC165D -> 74HC165
Connections:
- net BTN1 renamed BTN_LEFT
- net BTN2 renamed BTN_UP
- net BTN3 renamed BTN_RIGHT
- net BTN4 renamed BTN_DOWN
- net BTN5 renamed BTN_Y
- net BTN6 renamed BTN_X
- net BTN7 renamed BTN_L_BUMP
- net BTN8 renamed BTN_R_BUMP
Routing:
- net Vneo: track 96.4 -> 64.9 mm
- net PL/DATA: track 55.0 -> 44.8 mm
- net Net-(D4-DOUT): track 7.92 -> 0.00 mm
- net Net-(D3-DOUT): track 7.92 -> 0.00 mm
- net Net-(D2-DOUT): track 7.92 -> 0.00 mm
- net Net-(D1-DOUT): track 7.92 -> 0.00 mm
- net Net-(D1-DIN): track 7.52 -> 0.00 mm
- net SER: track 40.3 -> 41.5 mm
- net GND: vias 4 -> 3
Other:
- board text added: "v0.5"
- board text removed: "LED0"
- board text removed: "LED1"
- board text removed: "LED2"
- board text removed: "LED3"
- board text removed: "LED4"
- board text removed: "v0.6"

Commit message: Updated gitignore, removed spurious DS_Store and removed neopixel busbar
Routing:
- net Vneo: track 64.9 -> 30.7 mm
Changed lines of the file:
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@@
 				(font
 					(size 1.27 1.27)
+					(thickness 0.15)
 				)
 			)
@@
 				(font
 					(size 1.27 1.27)
+					(thickness 0.15)
 				)
 			)
@@
 				(font
 					(size 1.27 1.27)
+					(thickness 0.15)
 				)
 			)
@@
 				(font
 					(size 1.27 1.27)
+					(thickness 0.15)
 				)
 				(justify mirror)
@@
 				(font
 					(size 1.27 1.27)
+					(thickness 0.15)
 				)
 				(justify mirror)
@@
 				(font
 					(size 1.27 1.27)
+					(thickness 0.15)
 				)
 				(justify mirror)
@@
 				(font
 					(size 1.27 1.27)
+					(thickness 0.15)
 				)
 			)
@@
 				(font
 					(size 1.27 1.27)
+					(thickness 0.15)
 				)
 				(justify mirror)
@@
 				(font
 					(size 1.27 1.27)
+					(thickness 0.15)
 				)
 				(justify mirror)
@@
 				(font
 					(size 1.27 1.27)
+					(thickness 0.15)
 				)
 				(justify mirror)
@@
 				(font
 					(size 1.27 1.27)
+					(thickness 0.15)
 				)
 				(justify mirror)
@@
 				(font
 					(size 1.27 1.27)
+					(thickness 0.15)
 				)
 				(justify mirror)
@@
 				(font
 					(size 1.27 1.27)
+					(thickness 0.15)
 				)
 			)
@@
 				(font
 					(size 1.27 1.27)
+					(thickness 0.15)
 				)
 				(justify mirror)
@@
 				(font
 					(size 1.27 1.27)
+					(thickness 0.15)
 				)
 				(justify mirror)
@@
 				(polygon
 					(pts
-						(xy 81.827773 74.299002) (xy 82.955443 74.299002) (xy 82.955443 73.830055) (xy 81.827773 73.830055)
+						(xy 81.451151 74.111423) (xy 83.023586 74.111423) (xy 83.023586 73.548688) (xy 81.451151 73.548688)
 					)
 				)
@@
 				(polygon
 					(pts
-						(xy 81.377128 63.001549) (xy 82.170673 63.001549) (xy 82.170673 63.802421) (xy 82.586863 63.802421)
-						(xy 82.586863 63.001549) (xy 83.384804 63.001549) (xy 83.384804 62.583161) (xy 82.586863 62.583161)
-						(xy 82.586863 61.785952) (xy 82.170673 61.785952) (xy 82.170673 62.583161) (xy 81.377128 62.583161)
+						(xy 80.664183 62.911423) (xy 81.762543 62.911423) (xy 81.762543 63.99) (xy 82.327477 63.99) (xy 82.327477 62.911423)
+						(xy 83.425837 62.911423) (xy 83.425837 62.348688) (xy 82.327477 62.348688) (xy 82.327477 61.270111)
+						(xy 81.762543 61.270111) (xy 81.762543 62.348688) (xy 80.664183 62.348688)
 					)
 				)
@@
 	)
 	(segment
-		(start 120.164719 65.664719)
-		(end 118.6 65.664719)
-		(width 0.5)
-		(layer "F.Cu")
-		(net 28)
-	)
-	(segment
-		(start 94.564719 65.6)
-		(end 94.5 65.664719)
-		(width 0.25)
-		(layer "F.Cu")
-		(net 28)
-	)
-	(segment
-		(start 118.564719 65.629438)
-		(end 118.6 65.664719)
-		(width 0.25)
-		(layer "F.Cu")
-		(net 28)
-	)
-	(segment
 		(start 110.5 77)
 		(end 113 74.5)
@@
 	)
 	(segment
-		(start 118.6 65.664719)
-		(end 110.6 65.664719)
-		(width 0.5)
-		(layer "F.Cu")
-		(net 28)
-	)
-	(segment
-		(start 102.564719 65.529438)
-		(end 102.7 65.664719)
-		(width 0.25)
-		(layer "F.Cu")
-		(net 28)
-	)
-	(segment
 		(start 110.5 79)
 		(end 110.5 77)
@@
 	)
 	(segment
-		(start 110.564719 65.629438)
-		(end 110.6 65.664719)
-		(width 0.25)
-		(layer "F.Cu")
-		(net 28)
-	)
-	(segment
-		(start 121.5 67)
-		(end 120.164719 65.664719)
-		(width 0.5)
-		(layer "F.Cu")
-		(net 28)
-	)
-	(segment
-		(start 94.5 65.664719)
-		(end 88.235281 65.664719)
-		(width 0.5)
-		(layer "F.Cu")
-		(net 28)
-	)
-	(segment
 		(start 113 72.5)
 		(end 113 72)
@@
 	)
 	(segment
-		(start 102.7 65.664719)
-		(end 94.5 65.664719)
-		(width 0.5)
-		(layer "F.Cu")
-		(net 28)
-	)
-	(segment
 		(start 114.25 70.75)
 		(end 120 70.75)
@@
 	)
 	(segment
-		(start 110.6 65.664719)
-		(end 102.7 65.664719)
-		(width 0.5)
-		(layer "F.Cu")
-		(net 28)
-	)
-	(segment
 		(start 121.5 69.25)
 		(end 121.5 67)
@@
 			(thermal_bridge_width 0.2)
 			(island_removal_mode 2)
-			(island_area_min 10)
+			(island_area_min 15)
 		)
 		(polygon
